File: DualPedalBoardAmpSt.sch (KiCad schematic (older format))
At the start: 42 parts, among them J1 R-IN, J2 DC_IN, J3 out, J4 L-IN, J5 L-OUT, SW1 SDBY_MUTE, U1 TDA7293, U2 TDA7293, U3 TDA7293, U4 TDA7293

Commit message: improve design
Parts:
- U1, U2, U3, U4: symbol Amplifier_Audio:TDA7293 -> DualPedalBoardAmpSt-rescue:TDA7293-Amplifier_Audio
Changed lines of the file:
@@
 $EndDescr
 $Comp
-L Amplifier_Audio:TDA7293 U1
+L DualPedalBoardAmpSt-rescue:TDA7293-Amplifier_Audio U1
 U 1 1 5D589487
 P 3750 2450
@@
 $EndComp
 $Comp
-L Amplifier_Audio:TDA7293 U2
+L DualPedalBoardAmpSt-rescue:TDA7293-Amplifier_Audio U2
 U 1 1 5D63CB1F
 P 9000 2350
@@
 	3500 5600 3500 5550
 $Comp
-L Amplifier_Audio:TDA7293 U3
+L DualPedalBoardAmpSt-rescue:TDA7293-Amplifier_Audio U3
 U 1 1 5FE134F1
 P 3800 5100
@@
 	8800 5500 8800 5450
 $Comp
-L Amplifier_Audio:TDA7293 U4
+L DualPedalBoardAmpSt-rescue:TDA7293-Amplifier_Audio U4
 U 1 1 602D760F
 P 9100 5000
